File: Esquemático/schematic_robot/schematic_robot.kicad_sch (KiCad schematic)
At the start: 27 parts, among them M1 Motor_Servo, M2 Motor_Servo, M3 Motor_Servo, M4 Motor_Servo, M5 Motor_Servo, M6 Stepper_Motor_bipolar, Q1 PMOS, U1 TB6600, U2 ESP32-WROOM-32, U3 PCA9685PW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

Commit message: datasheet + kicad
datasheet + kicad
Parts:
- removed BT1: Battery 12V, symbol Device:Battery
- removed C1, C2, C3, C4, C5: 470uF, symbol Device:C_Polarized
- removed C10, C6, C7, C8, C9: 0.1uF, symbol Device:C
- removed D1: D_Zener, symbol Device:D_Zener_Filled
- removed M6: Stepper_Motor_bipolar, symbol Motor:Stepper_Motor_bipolar
- removed Q1: PMOS, symbol Simulation_SPICE:PMOS
- removed R3: 100k, symbol Device:R
- removed U4, U5: XL4015, Package_TO_SOT_SMD:TO-263-5_TabPin3, symbol Regulator_Switching:XL4015
- added J1: Conn_01x04_Pin, symbol Connector:Conn_01x04_Pin
- added J2, J3, J4, J5, J6, J7, J8, J9: Conn_01x01_Socket, symbol Connector:Conn_01x01_Socket
Connections:
- net +12V: now also J2.1 (Pin_1), J6.1 (Pin_1)
- net GND: now also J4.1 (Pin_1), J9.1 (Pin_1); no longer U1.1 (ENA-), U1.11 (GND), U1.3 (DIR-), U1.5 (PUL-)
- net at U2.2 (VDD): now also J8.1 (Pin_1)
- net at M1.2 (+), M2.2 (+), M3.2 (+)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: now also J3.1 (Pin_1)
- net at U1.8 (B+): now also J1.1 (Pin_1)
- net at U1.7 (B-): now also J1.2 (Pin_2)
- net at U1.9 (A-): now also J1.3 (Pin_3)
- net at U1.10 (A+): now also J1.4 (Pin_4)
- new net Earth: J5.1 (Pin_1), J7.1 (Pin_1), U1.1 (ENA-), U1.11 (GND), U1.3 (DIR-), U1.5 (PUL-)
- no-connect marks 50 -> 46
