File: Esquemático/schematic_robot/schematic_robot.kicad_sch (KiCad schematic)
At the start: 19 parts, among them J1 Conn_01x04_Pin, J2 Conn_01x01_Socket, J3 Conn_01x01_Socket, J4 Conn_01x01_Socket, J5 Conn_01x01_Socket, J6 Conn_01x01_Socket, J7 Conn_01x01_Socket, J8 Conn_01x01_Socket, J9 Conn_01x01_Socket, M1 Motor_Servo, M2 Motor_Servo, M3 Motor_Servo, M4 Motor_Servo, M5 Motor_Servo, U1 TB6600, U2 ESP32-WROOM-32, U3 PCA9685PW

Commit message: atualizei uns trem
esquema
Parts:
- J1: footprint (none) -> Connector_PinSocket_2.54mm:PinSocket_1x04_P2.54mm_Vertical
- J2, J3, J4, J5, J6, J7, J8, J9: footprint (none) -> Connector_PinSocket_2.54mm:PinSocket_1x01_P2.54mm_Vertical
- M1, M2, M3, M4, M5: footprint (none) -> Connector_JST:JST_EH_B3B-EH-A_1x03_P2.50mm_Vertical
- R1, R2: footprint (none) -> Resistor_THT:R_Axial_DIN0207_L6.3mm_D2.5mm_P10.16mm_Horizontal
- U1: footprint (none) -> Connector_PinSocket_2.54mm:PinSocket_1x12_P2.54mm_Vertical
Other:
- moved on the sheet: J1, J2, J3, J4, J5, J6, J7, J8, J9, M1, M2, M3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

Commit message: MUDEI MAIS
AOBA
Connections:
- net +5V is gone; now on net 5V: R1.1, R2.1, U3.14 (VSS)
- net 5V: now reaches J3.1 (Pin_1), M1.2 (+), M2.2 (+), M3.2 (+), M4.2 (+), M5.2 (+)
- net 5V: now also J8.1 (Pin_1), U2.2 (VDD)
- net +12V renamed 12V
Other:
- note removed: "+5V"

Commit message: Upload da luva
Parts:
- added Q1: BSS138, Package_TO_SOT_SMD:SOT-23, symbol Transistor_FET:BSS138
- added R3, R4: 10k, symbol Device:R
Connections:
- net 5V: now also R4.1
- new net 3.3V: Q1.1 (G), R3.1
- new net HIGH_SIDE_LOGICAL_OUTPUT: Q1.3 (D), R4.2
- new net LOW_SIDE_LOGICAL_OUTPUT: Q1.2 (S), R3.2
Other:
- moved on the sheet: J1, U1

Commit message: Correção final
Parts:
- removed Q1: BSS138, Package_TO_SOT_SMD:SOT-23, symbol Transistor_FET:BSS138
- removed R3, R4: 10k, symbol Device:R
- added C1, C5: 220uF, symbol Device:C_Polarized_US
- added C2, C3, C4: 105uF, symbol Device:C
- added D1: B540, symbol Device:D_Zener_Filled
- added J10, J11, J12, J13: Conn_01x01_Socket, Connector_PinSocket_2.54mm:PinSocket_1x01_P2.54mm_Vertical, symbol Connector:Conn_01x01_Socket
- added L1: 47uH, symbol Device:L
- added R3, R4: R_Variable, symbol Device:R_Variable
- added U4: XL4015, Package_TO_SOT_SMD:TO-263-5_TabPin3, symbol Regulator_Switching:XL4015
Connections:
- net 12V: now also J12.1 (Pin_1)
- net 5V: now also U2.3 (EN)
- net Earth: now also J11.1 (Pin_1)
- net GND: now also U3.1 (A0), U3.2 (A1), U3.23 (~{OE}), U3.24 (A5), U3.3 (A2), U3.4 (A3), U3.5 (A4), C1.2, C2.2, C4.2, C5.2, D1.2 (A), J13.1 (Pin_1), R3.2, U4.1 (GND)
- new net: D1.1 (K), L1.1, U4.3 (SW)
- new net: C3.2, U4.4 (VC)
- new net: C4.1, C5.1, L1.2, R4.1
- new net Battery : J10.1 (Pin_1)
- new net Vin: C1.1, C2.1, C3.1, U4.5 (VIN)
- new net Vout: R3.1, R4.2, U4.2 (FB)
- no-connect marks 46 -> 39
Other:
- note added: "Tensão da bateria regulada"
- note added: "Vout = 1.25*(1+R4/R3)"
- moved on the sheet: J1, J6, J7, J8, J9, U1, U2

Commit message: Atualização do esquemático e datasheets, exclusão da pasta src
Parts:
- removed C1, C5: 220uF, symbol Device:C_Polarized_US
- removed D1: B540, symbol Device:D_Zener_Filled
- removed J1: Conn_01x04_Pin, Connector_PinSocket_2.54mm:PinSocket_1x04_P2.54mm_Vertical, symbol Connector:Conn_01x04_Pin
- removed J10, J11, J12, J13, J2, J3, J4, J5, J6, J7, J8, J9: Conn_01x01_Socket, Connector_PinSocket_2.54mm:PinSocket_1x01_P2.54mm_Vertical, symbol Connector:Conn_01x01_Socket
- removed L1: 47uH, symbol Device:L
- removed R3, R4: R_Variable, symbol Device:R_Variable
- removed U4: XL4015, Package_TO_SOT_SMD:TO-263-5_TabPin3, symbol Regulator_Switching:XL4015
- added C1, C10, C12, C14, C6, C8: 0.33uF, Capacitor_THT:CP_Radial_Tantal_D4.5mm_P2.50mm, symbol Device:C
- added C11, C13, C15, C7, C9: 0.1uF, Capacitor_THT:CP_Radial_Tantal_D4.5mm_P2.50mm, symbol Device:C
- added C16: 10uF, symbol Device:C
- added C5: 10uF, Capacitor_THT:CP_Radial_Tantal_D4.5mm_P2.50mm, symbol Device:C
- added J1: Jack-DC, symbol Connector:Jack-DC
- added M6: Stepper_Motor_bipolar, TerminalBlock:TerminalBlock_bornier-2_P5.08mm, symbol Motor:Stepper_Motor_bipolar
- added M7: Motor_DC, TerminalBlock:TerminalBlock_bornier-2_P5.08mm, symbol Motor:Motor_DC
- added R10, R11, R12, R13, R14, R8, R9: 10k, Resistor_THT:R_Array_SIP5, symbol Device:R
- added R3, R4, R5, R6, R7: 200ohms, Resistor_THT:R_Array_SIP5, symbol Device:R
- added U10, U4, U6, U7, U8, U9: LM7805_TO220, Package_TO_SOT_THT:TO-220-3_Vertical, symbol Regulator_Linear:LM7805_TO220
- added U11: LM1117DT-3.3, Package_TO_SOT_SMD:TO-252-3_TabPin2, symbol Regulator_Linear:LM1117DT-3.3
- added U5: L298N, Package_TO_SOT_THT:TO-220-15_P2.54x2.54mm_StaggerOdd_Lead4.58mm_Vertical, symbol Driver_Motor:L298N
- C2: value 105uF -> 0.1uF; footprint (none) -> Capacitor_THT:CP_Radial_Tantal_D4.5mm_P2.50mm
- C3: value 105uF -> 100nF; footprint (none) -> Capacitor_THT:CP_Radial_Tantal_D4.5mm_P2.50mm
- C4: value 105uF -> 100uF; footprint (none) -> Capacitor_THT:CP_Radial_Tantal_D4.5mm_P2.50mm
- R1: value 4.7k -> 121ohms; footprint Resistor_THT:R_Axial_DIN0207_L6.3mm_D2.5mm_P10.16mm_Horizontal -> Resistor_THT:R_Array_SIP5
- R2: value 4.7k -> 1k; footprint Resistor_THT:R_Axial_DIN0207_L6.3mm_D2.5mm_P10.16mm_Horizontal -> Resistor_THT:R_Array_SIP5
- renumbered M4 to M2, M2 to M4
Connections:
- net Earth is gone; now on net GND: U1.1 (ENA-), U1.11 (GND), U1.3 (DIR-), U1.5 (PUL-)
- net 5V: now also U5.6 (EnA); no longer M1.2 (+), M2.2 (+), M3.2 (+), M4.2 (+), M5.2 (+), R1.1, R2.1, U2.2 (VDD), U2.3 (EN), U3.14 (VSS)
- net GND: now also C3.2, R2.2, U3.14 (VSS), C1.2, C10.2, C11.2, C12.2, C13.2, C14.2, C15.2, C16.1, C5.2, C6.2, C7.2, C8.2, C9.2, J1.2, R14.1, U10.2 (GND), U4.2 (GND), U5.8 (GND), U6.2 (GND), U7.2 (GND), U8.2 (GND), U9.2 (GND); no longer U3.1 (A0), U3.2 (A1), U3.23 (~{OE}), U3.24 (A5), U3.25 (EXTCLK), U3.28 (VDD), U3.3 (A2), U3.4 (A3), U3.5 (A4)
- net PWM1: now also R3.2; no longer U3.6 (LED0)
- net PWM2: now also M2.1 (PWM), R4.2; no longer M4.1 (PWM), U3.7 (LED1)
- net PWM3: now also R5.2; no longer U3.8 (LED2)
- net PWM4: now also M4.1 (PWM), R6.2; no longer M2.1 (PWM), U3.9 (LED3)
- net PWM5: now also R7.2; no longer U3.10 (LED4)
- net SCL: no longer R2.2
- net SDA: no longer R1.2
- net at U1.8 (B+): now also M6.4
- net at U1.7 (B-): now also M6.3
- net at U1.9 (A-): now also M6.1
- net at U1.10 (A+): now also M6.2 (-)
- net 3.3V: now reaches C4.1
- net 3.3V: now also R1.1, U2.2 (VDD), U3.28 (VDD), C16.2, R10.1, R11.1, R12.1, R13.1, R8.1, R9.1, U11.2 (VO)
- net DC_Motor(+): now reaches U2.8 (IO32)
- net DC_Motor(+): now also U5.5 (IN1)
- net DC_Motor(-): now reaches U2.9 (IO33)
- net DC_Motor(-): now also U5.7 (IN2)
- net 12V renamed +12V
- net +12V: now also C1.1, C10.1, C12.1, C14.1, C6.1, C8.1, J1.1, U10.1 (VI), U4.1 (VI), U5.4 (Vs), U6.1 (VI), U7.1 (VI), U8.1 (VI), U9.1 (VI)
- net Vin: no longer names the net of C3.1
- net Vin: now also R1.2, R2.1, U11.1 (GND); no longer C2.1
- new net: R6.1, U3.9 (LED3)
- new net: R3.1, U3.6 (LED0)
- new net: R13.2, U3.24 (A5)
- new net: R5.1, U3.8 (LED2)
- new net: R8.2, U3.1 (A0)
- new net: R14.2, U3.23 (~{OE}), U3.25 (EXTCLK)
- new net: R4.1, U3.7 (LED1)
- new net: M7.1 (+), U5.2 (OUT1)
- new net: M7.2 (-), U5.3 (OUT2)
- new net: R7.1, U3.10 (LED4)
- new net: R9.2, U3.2 (A1)
- new net: R10.2, U3.3 (A2)
- new net: R11.2, U3.4 (A3)
- new net: R12.2, U3.5 (A4)
- new net +5V: C2.1, C5.1, U11.3 (VI), U4.3 (VO), U5.9 (Vss)
- new net +5V1: C11.1, M1.2 (+), U8.3 (VO)
- new net +5V2: C7.1, M2.2 (+), U6.3 (VO)
- new net +5V3: C13.1, M3.2 (+), U9.3 (VO)
- new net +5V4: C9.1, M4.2 (+), U7.3 (VO)
- new net +5V5: C15.1, M5.2 (+), U10.3 (VO)
- no-connect marks 39 -> 44
Other:
- note added: "0.5A"
- note added: "10mA"
- note added: "36mA"
- note added: "3A"
- note added: "4.5A"
- note added: "LM7805: Voltage Supply 12V Voltage Output 5V Max Current Output 1A"
- note added: "Ponte H com motor DC"
- note added: "Regulador 12V para 5V"
- note added: "Servo motor: Voltage Supply = 5V Current Supply = 0.5A ~ 0.9A"
- note removed: "Tensão da bateria regulada"
- note removed: "Vout = 1.25*(1+R4/R3)"
- moved on the sheet: M1, M2, M3, M4, M5, U1, U2, U3
