File: Esquemático/schematic_glove/schematic_glove.kicad_sch (KiCad schematic)
At the start: 4 parts, among them J1 Conn_01x02_Socket, J3 Conn_01x04_Socket, U1 ESP32-S3-WROOM-1

Commit message: Esquemático com fonte e substituição de mcu
Parts:
- removed U1: ESP32-S3-WROOM-1, RF_Module:ESP32-S3-WROOM-1, symbol RF_Module:ESP32-S3-WROOM-1
- added J2, J4, J5, J6: Conn_01x01_Socket, Connector_PinSocket_2.54mm:PinSocket_1x01_P2.54mm_Vertical, symbol Connector:Conn_01x01_Socket
- added U2: ESP32-WROOM-32, RF_Module:ESP32-WROOM-32, symbol RF_Module:ESP32-WROOM-32
Connections:
- net 3.3V: now also J3.1 (Pin_1), J5.1 (Pin_1), U2.2 (VDD)
- net 5V: now also J2.1 (Pin_1); no longer J3.1 (Pin_1)
- net GND: now also J6.1 (Pin_1), U2.1 (GND), U2.15 (GND), U2.38 (GND), U2.39 (GND)
- net PWM: now also U2.27 (IO16)
- net SCL: now also U2.36 (IO22)
- net SDA: now also U2.33 (IO21)
- new net Earth: J4.1 (Pin_1)
- no-connect marks 0 -> 30
Other:
- note added: "ESP32-WROOM-32"
- note added: "POWER SUPPLY"
- note removed: "MINI ESP32"
- moved on the sheet: J1, J3, R1
